Commit message: Balanced on wheels

File: description/robot_core.xacro (robot description, xacro)
@@ -18,9 +18,9 @@
     <parent link="base_link"/>
     <child link="chassis" />
-    <origin xyz="-0.2 0 0.075"/>
+    <origin xyz="-0.2 0 0.05"/>
 </joint>
 <link name="chassis">
 <visual>
-    <origin xyz="0.2 0 0" />
+    <origin xyz="0.2 0 0.075" />
     <geometry>
         <box size ="0.4 0.4 0.15" />
@@ -41,5 +41,5 @@
     <parent link="base_link"/>
     <child link="left_wheel"/>
-    <origin xyz="0 0.3 0.075"/>
+    <origin xyz="0 0.22 0.05"/>
     <axis xyz="0 1 0" />
 </joint>
@@ -56,5 +56,5 @@
     <parent link="base_link"/>
     <child link="right_wheel"/>
-    <origin xyz="0 -0.3 0.075"/>
+    <origin xyz="0 -0.22 0.05"/>
     <axis xyz="0 1 0" />
 </joint>

Commit message: Casterwheel updated

File: description/robot_core.xacro (robot description, xacro)
@@ -59,3 +59,16 @@
     <axis xyz="0 1 0" />
 </joint>
+<joint name ="caster_wheel_joint" type="fixed">
+    <parent link="chassis"/>
+    <child link="caster_wheel" />
+    <origin xyz="0.24 0 0.045" />
+</joint>
+<link name="caster_wheel">
+<visual>
+    <geometry>
+        <sphere radius="0.095"/>
+    </geometry>
+    <material name="black"/>
+</visual>
+</link>
 </robot>

Commit message: Inertial and mass values added

File: description/robot_core.xacro (robot description, xacro)
@@ -1,4 +1,5 @@
 <?xml version="1.0"?>
 <robot xmlns:xacro="http://www.ros.org/wiki/xacro"  name="robot">
+<xacro:include filename="inertia_macro.xacro"/>
 <material name="white">
     <color rgba = "1 1 1 1"/>
@@ -28,5 +29,20 @@
     <material name="white" />
 </visual>
+<collision>
+    <origin xyz="0.2 0 0.075" />
+    <geometry>
+        <box size ="0.4 0.4 0.15" />
+    </geometry>
+</collision>
+<xacro:inertial_box mass="0.5" x="0.4" y="0.4" z="0.15">
+    <origin xyz="0.2 0 0.075" rpy="0 0 0"/>
+</xacro:inertial_box>
 </link>
+<joint name="wheel_link" type="continuous">
+    <parent link="base_link"/>
+    <child link="left_wheel"/>
+    <origin xyz="0 0.22 0.05"/>
+    <axis xyz="0 1 0" />
+</joint>
 <link name="left_wheel">
 <visual>
@@ -37,11 +53,14 @@
     <material name="black"/>
 </visual>
+<collision>
+    <origin xyz="0 0 0" rpy="1.5708 0 0"/>
+    <geometry>
+        <cylinder radius="0.05" length="0.04"/>
+    </geometry>
+</collision>
+<xacro:inertial_cylinder mass="0.1" length="0.04" radius="0.05">
+    <origin xyz="0 0 0" rpy="1.5708 0 0"/>
+</xacro:inertial_cylinder>
 </link>
-<joint name="wheel_link" type="continuous">
-    <parent link="base_link"/>
-    <child link="left_wheel"/>
-    <origin xyz="0 0.22 0.05"/>
-    <axis xyz="0 1 0" />
-</joint>
 <link name="right_wheel">
 <visual>
@@ -52,4 +71,13 @@
     <material name="black"/>
 </visual>
+<collision>
+    <origin xyz="0 0 0" rpy="1.5708 0 0"/>
+    <geometry>
+        <cylinder radius="0.05" length="0.04" />
+    </geometry>
+</collision>
+<xacro:inertial_cylinder mass="0.1" length="0.04" radius="0.05">
+    <origin xyz="0 0 0" rpy="1.5708 0 0" />
+</xacro:inertial_cylinder>
 </link>
 <joint name="right_wheel_joint" type="continuous">
@@ -66,4 +94,5 @@
 <link name="caster_wheel">
 <visual>
+    <origin xyz="0 0 0" rpy="0 0 0"/>
     <geometry>
         <sphere radius="0.095"/>
@@ -71,4 +100,13 @@
     <material name="black"/>
 </visual>
+<collision>
+    <origin xyz="0 0 0" rpy="0 0 0"/>
+    <geometry>
+        <sphere radius="0.095"/>
+    </geometry>
+</collision>
+<xacro:inertial_sphere mass="0.1" radius="0.095">
+    <origin xyz="0 0 0" rpy="0 0 0" />
+</xacro:inertial_sphere>
 </link>
 </robot>
