Commit message: Control systems added

File: description/robot.urdf.xacro (robot description, xacro)
@@ -2,3 +2,4 @@
 <robot xmlns:xacro="http://www.ros.org/wiki/xacro"  name="robot">
    <xacro:include filename="robot_core.xacro" />
+   <xacro:include filename="gazebo_control.xacro" />
 </robot>

File: description/robot_core.xacro (robot description, xacro)
@@ -39,5 +39,12 @@
 </xacro:inertial_box>
 </link>
-<joint name="wheel_link" type="continuous">
+<gazebo reference = "chassis">
+<visual><material>
+    <ambient>1 1 1 1</ambient>
+    <diffuse>1 1 1 1</diffuse>
+    <specular>1 1 1 1</specular>
+</material></visual>
+</gazebo>
+<joint name="left_wheel_joint" type="continuous">
     <parent link="base_link"/>
     <child link="left_wheel"/>
@@ -63,4 +70,17 @@
 </xacro:inertial_cylinder>
 </link>
+<gazebo reference="left_wheel">
+<visual><material>
+    <ambient>0 0 0 1</ambient>
+    <diffuse>0 0 0 1</diffuse>
+    <specular>0 0 0 1</specular>
+</material></visual>
+</gazebo>
+<joint name="right_wheel_joint" type="continuous">
+    <parent link="base_link"/>
+    <child link="right_wheel"/>
+    <origin xyz="0 -0.22 0.05"/>
+    <axis xyz="0 1 0" />
+</joint>
 <link name="right_wheel">
 <visual>
@@ -81,10 +101,11 @@
 </xacro:inertial_cylinder>
 </link>
-<joint name="right_wheel_joint" type="continuous">
-    <parent link="base_link"/>
-    <child link="right_wheel"/>
-    <origin xyz="0 -0.22 0.05"/>
-    <axis xyz="0 1 0" />
-</joint>
+<gazebo reference="right_wheel">
+<visual><material>
+    <ambient>0 0 0 1</ambient>
+    <diffuse>0 0 0 1</diffuse>
+    <specular>0 0 0 1</specular>
+</material></visual>
+</gazebo>
 <joint name ="caster_wheel_joint" type="fixed">
     <parent link="chassis"/>
@@ -110,3 +131,10 @@
 </xacro:inertial_sphere>
 </link>
+<gazebo reference="caster_wheel">
+<visual><material>
+    <ambient>0.2 0.2 1 1</ambient>
+    <diffuse>0.2 0.2 1 1</diffuse>
+    <specular>0.2 0.2 1 1</specular>
+</material></visual>
+</gazebo>
 </robot>

Commit message: Changes

File: description/robot.urdf.xacro (robot description, xacro)
@@ -1,5 +1,7 @@
 <?xml version="1.0"?>
-<robot xmlns:xacro="http://www.ros.org/wiki/xacro"  name="robot">
-   <xacro:include filename="robot_core.xacro" />
-   <xacro:include filename="gazebo_control.xacro" />
+<robot xmlns:xacro="http://www.ros.org/wiki/xacro" name="robot">
+  <xacro:include filename="robot_core.xacro"/>
+  <xacro:include filename="gazebo_control.xacro"/>
+  <xacro:include filename="ros2_control.xacro"/>
+  <xacro:my_bot_ros2_control/>
 </robot>

File: description/robot_core.xacro (robot description, xacro)
@@ -111,5 +111,5 @@
     <parent link="chassis"/>
     <child link="caster_wheel" />
-    <origin xyz="0.24 0 0.045" />
+    <origin xyz="0.25 0 0.045" />
 </joint>
 <link name="caster_wheel">
@@ -140,3 +140,43 @@
 <mu2 value="0.001"/>
 </gazebo>
+<joint name="dvl_joint" type="fixed">
+    <parent link="chassis"/>
+    <child link="dvl_link"/>
+    <origin xyz="0.05 0 -0.01" rpy="0 0 0"/>
+</joint>
+<link name="dvl_link">
+<visual>
+    <origin xyz="0 0 0" rpy="0 0 0"/>
+    <geometry>
+        <cylinder radius="0.03" length="0.03"/>
+    </geometry>
+    <material name="blue" />
+</visual>
+<collision>
+    <origin xyz="0 0 0" rpy="0 0 0"/>
+    <geometry>
+        <cylinder radius="0.03" length="0.03" />
+    </geometry>
+</collision>
+</link>
+<joint name="dvl_frame_joint" type="fixed">
+    <parent link="dvl_link"/>
+    <child link="dvl_frame"/>
+    <origin xyz="0 0 0" rpy="0 3.14159 0"/>
+</joint>
+<link name="dvl_frame">
+<visual>
+    <origin xyz="0 0 0" rpy="0 0 0"/>
+    <geometry>
+        <cylinder radius="0.03" length="0.015"/>
+    </geometry>
+    <material name="white"/>
+</visual>
+<collision>
+    <origin xyz="0 0 0" rpy="0 0 0"/>
+    <geometry>
+        <cylinder radius="0.03" length="0.015"/>
+    </geometry>
+</collision>
+</link>
 </robot>
